File: eagle/Timelapse.brd (EAGLE design)
At the start: 47.9 x 33 mm, 11 parts, among them U1 ATTINY2313V-10PU, X1 1501_04

Commit message: updated eagle with small changes
-move jumper
-rearrange diagram
Parts:
- moved JP1 1.27 mm to (2.54, 20.3)
Routing:
- net N$11: track 17.8 -> 19.0 mm
- net N$9: track 69.0 -> 70.3 mm
Changed lines of the file:
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@@
 <attribute name="OC_FARNELL" value="1216977" x="44.45" y="22.86" size="1.778" layer="27" rot="R270" display="off"/>
 </element>
-<element name="JP1" library="jumper" package="JP1" value="Battery" x="3.81" y="20.32" rot="R90"/>
+<element name="JP1" library="jumper" package="JP1" value="Battery" x="2.54" y="20.32" rot="R90"/>
 <element name="LED1" library="display-kingbright" package="SA39-11SRWA" value="7-SEG_SA39-11SRWA" x="6.35" y="39.37">
 <attribute name="OC_NEWARK" value="unknown" x="6.35" y="39.37" size="1.778" layer="27" display="off"/>
@@
 <contactref element="U1" pad="3"/>
 <contactref element="LED1" pad="9"/>
-<wire x1="10.16" y1="41.91" x2="13.97" y2="41.91" width="0.4064" layer="16"/>
-<wire x1="13.97" y1="41.91" x2="13.97" y2="39.37" width="0.4064" layer="16"/>
-<wire x1="13.97" y1="39.37" x2="17.78" y2="39.37" width="0.4064" layer="16"/>
+<wire x1="10.16" y1="41.91" x2="12.7" y2="41.91" width="0.4064" layer="16"/>
+<wire x1="12.7" y1="41.91" x2="12.7" y2="39.37" width="0.4064" layer="16"/>
+<wire x1="12.7" y1="39.37" x2="17.78" y2="39.37" width="0.4064" layer="16"/>
 </signal>
 <signal name="N$3">
@@
 <wire x1="2.54" y1="27.94" x2="0.29" y2="27.94" width="0.4064" layer="16"/>
 <wire x1="0.29" y1="27.94" x2="0.29" y2="29.92" width="0.4064" layer="16"/>
-<wire x1="2.54" y1="20.32" x2="2.54" y2="27.94" width="0.4064" layer="16"/>
 <wire x1="25.4" y1="44.45" x2="24.13" y2="44.45" width="0.4064" layer="16"/>
 <wire x1="24.13" y1="44.45" x2="24.13" y2="25.4" width="0.4064" layer="16"/>
@@
 <wire x1="13.97" y1="26.67" x2="13.97" y2="31.75" width="0.4064" layer="16"/>
 <wire x1="13.97" y1="31.75" x2="2.54" y2="31.75" width="0.4064" layer="16"/>
-<wire x1="2.54" y1="31.75" x2="2.54" y2="27.94" width="0.4064" layer="16"/>
+<wire x1="2.54" y1="31.75" x2="2.54" y2="29.21" width="0.4064" layer="16"/>
+<wire x1="2.54" y1="29.21" x2="2.54" y2="27.94" width="0.4064" layer="16"/>
+<wire x1="1.27" y1="20.32" x2="1.27" y2="21.59" width="0.4064" layer="16"/>
+<wire x1="1.27" y1="21.59" x2="2.54" y2="21.59" width="0.4064" layer="16"/>
+<wire x1="2.54" y1="21.59" x2="2.54" y2="27.94" width="0.4064" layer="16"/>
 </signal>
 <signal name="N$10">
@@
 <wire x1="15.24" y1="25.4" x2="15.24" y2="24.13" width="0.4064" layer="16"/>
 <wire x1="15.24" y1="24.13" x2="17.78" y2="24.13" width="0.4064" layer="16"/>
-<wire x1="4.79" y1="29.92" x2="12.7" y2="29.92" width="0.4064" layer="16"/>
-<wire x1="12.7" y1="29.92" x2="12.7" y2="25.4" width="0.4064" layer="16"/>
-<wire x1="12.7" y1="25.4" x2="15.24" y2="25.4" width="0.4064" layer="16"/>
+<wire x1="4.79" y1="29.92" x2="11.43" y2="29.92" width="0.4064" layer="16"/>
+<wire x1="11.43" y1="29.92" x2="11.43" y2="25.4" width="0.4064" layer="16"/>
+<wire x1="11.43" y1="25.4" x2="15.24" y2="25.4" width="0.4064" layer="16"/>
 </signal>
 <signal name="N$11">
@@
 <contactref element="R1" pad="2"/>
 <contactref element="JP1" pad="1"/>
-<wire x1="5.08" y1="20.32" x2="7.62" y2="20.32" width="0.4064" layer="16"/>
+<wire x1="3.81" y1="20.32" x2="7.62" y2="20.32" width="0.4064" layer="16"/>
 <wire x1="7.62" y1="20.32" x2="7.62" y2="21.59" width="0.4064" layer="16"/>
 <wire x1="7.62" y1="22.86" x2="7.62" y2="25.4" width="0.4064" layer="16"/>
